File: Design/Eagle.smd/Modem.sch (EAGLE design)
At the start: 23 parts, among them Q1 BSS123

Commit message: Add input filter
Parts:
- added C4: 10uf, rcl:C-EUC1206
- added R12: 10k, rcl:R-EU_R0603
- C1: device eagle-ltspice:CC1206 -> eagle-ltspice:CC0603
- C3: value 1uf -> 220nf; device eagle-ltspice:CC1206 -> rcl:C-EUC0603
- R1, R2, R3, R4, R5, R6, R7, R8: device resistor:R-EU_R0805 -> resistor:R-EU_R0603
- R10, R11: value 100k -> 10k; device rcl:R-EU_R0805 -> rcl:R-EU_R0603
- R9: device rcl:R-EU_R0805 -> rcl:R-EU_R0603
Connections:
- new net N$10: C4.1, R10.2, R11.2, R12.2
- net A0: now also C3.1, R12.1; no longer C3.2, R10.2, R11.2
- net GND: now also C4.2
- net LINE_LEVEL_IN: now also C3.2; no longer C3.1
Other:
- moved on the sheet: C3, R9
